Commit message: tmp modifications

File: z1_description/urdf/z1.ros2_control.xacro (robot description, xacro)
@@ -9,8 +9,8 @@
         params="
         name:='z1'
-        sim_ignition:=true
+        sim_ignition:=false
         sim_coppelia:=false
         prefix:=''
-        with_gripper:=true
+        with_gripper:=false
         ">
         <ros2_control name="${name}" type="system">
@@ -29,10 +29,10 @@
             <joint name="joint1">
                 <command_interface name="position">
-                    <param name="min"> ${joint1_PositionMin} </param>
-                    <param name="max"> ${joint1_PositionMax} </param>
+                    <param name="min">${joint1_PositionMin}</param>
+                    <param name="max">${joint1_PositionMax}</param>
                 </command_interface>
                 <command_interface name="effort">
-                    <param name="min"> -${torqueMax} </param>
-                    <param name="max"> ${torqueMax} </param>
+                    <param name="min">-${torqueMax}</param>
+                    <param name="max">${torqueMax}</param>
                 </command_interface>
                 <state_interface name="position" />
@@ -42,11 +42,11 @@
             <joint name="joint2">
                 <command_interface name="position">
-                    <param name="min"> ${joint2_PositionMin} </param>
-                    <param name="max"> ${joint2_PositionMax} </param>
+                    <param name="min">${joint2_PositionMin}</param>
+                    <param name="max">${joint2_PositionMax}</param>
                 </command_interface>
                 <command_interface
                     name="effort">
-                    <param name="min"> -${torqueMax} </param>
-                    <param name="max"> ${torqueMax} </param>
+                    <param name="min">-${torqueMax}</param>
+                    <param name="max">${torqueMax}</param>
                 </command_interface>
                 <xacro:if value="${sim_ignition}">
@@ -64,10 +64,10 @@
             <joint name="joint3">
                 <command_interface name="position">
-                    <param name="min"> ${joint3_PositionMin} </param>
-                    <param name="max"> ${joint3_PositionMax} </param>
+                    <param name="min">${joint3_PositionMin}</param>
+                    <param name="max">${joint3_PositionMax}</param>
                 </command_interface>
                 <command_interface name="effort">
-                    <param name="min"> -${torqueMax} </param>
-                    <param name="max"> ${torqueMax} </param>
+                    <param name="min">-${torqueMax}</param>
+                    <param name="max">${torqueMax}</param>
                 </command_interface>
                 <xacro:if value="${sim_ignition}">
@@ -85,10 +85,10 @@
             <joint name="joint4">
                 <command_interface name="position">
-                    <param name="min"> ${joint4_PositionMin} </param>
-                    <param name="max"> ${joint4_PositionMax} </param>
+                    <param name="min">${joint4_PositionMin}</param>
+                    <param name="max">${joint4_PositionMax}</param>
                 </command_interface>
                 <command_interface name="effort">
-                    <param name="min"> -${torqueMax} </param>
-                    <param name="max"> ${torqueMax} </param>
+                    <param name="min">-${torqueMax}</param>
+                    <param name="max">${torqueMax}</param>
                 </command_interface>
                 <state_interface name="position" />
@@ -98,10 +98,10 @@
             <joint name="joint5">
                 <command_interface name="position">
-                    <param name="min"> ${joint5_PositionMin} </param>
-                    <param name="max"> ${joint5_PositionMax} </param>
+                    <param name="min">${joint5_PositionMin}</param>
+                    <param name="max">${joint5_PositionMax}</param>
                 </command_interface>
                 <command_interface name="effort">
-                    <param name="min"> -${torqueMax} </param>
-                    <param name="max"> ${torqueMax} </param>
+                    <param name="min">-${torqueMax}</param>
+                    <param name="max">${torqueMax}</param>
                 </command_interface>
                 <state_interface name="position" />
@@ -111,10 +111,10 @@
             <joint name="joint6">
                 <command_interface name="position">
-                    <param name="min"> ${joint6_PositionMin} </param>
-                    <param name="max"> ${joint6_PositionMax} </param>
+                    <param name="min">${joint6_PositionMin}</param>
+                    <param name="max">${joint6_PositionMax}</param>
                 </command_interface>
                 <command_interface name="effort">
-                    <param name="min"> -${torqueMax} </param>
-                    <param name="max"> ${torqueMax} </param>
+                    <param name="min">-${torqueMax}</param>
+                    <param name="max">${torqueMax}</param>
                 </command_interface>
                 <state_interface name="position" />
@@ -125,10 +125,10 @@
                 <joint name="jointGripper">
                     <command_interface name="position">
-                        <param name="min"> ${Gripper_PositionMin} </param>
-                        <param name="max"> ${Gripper_PositionMax} </param>
+                        <param name="min">${Gripper_PositionMin}</param>
+                        <param name="max">${Gripper_PositionMax}</param>
                     </command_interface>
                     <command_interface name="effort">
-                        <param name="min"> -${torqueMax} </param>
-                        <param name="max"> ${torqueMax} </param>
+                        <param name="min">-${torqueMax}</param>
+                        <param name="max">${torqueMax}</param>
                     </command_interface>
                     <state_interface name="position" />

File: z1_description/urdf/z1.urdf.xacro (robot description, xacro)
@@ -106,5 +106,5 @@
     </link>
     <joint name="joint3" type="revolute">
-        <origin rpy="0 0 0" xyz="-0.35 0 0" />
+        <origin rpy="0 -0.1 0" xyz="-0.35 0 0" />
         <parent link="link02" />
         <child link="link03" />
@@ -306,6 +306,6 @@
         <gazebo reference="world" />
         <gazebo>
-            <plugin filename="libign_ros2_control-system.so"
-                name="ign_ros2_control::IgnitionROS2ControlPlugin">
+            <!-- <plugin filename="libign_ros2_control-system.so" name="ign_ros2_control::IgnitionROS2ControlPlugin"> -->
+            <plugin filename="libgz_ros2_control-system.so" name="gz_ros2_control::GazeboSimROS2ControlPlugin">
                 <parameters> $(arg controllers) </parameters>
                 <robot_param> robot_description </robot_param>

Commit message: Revert "tmp modifications"
This reverts commit 35dd2050125ba4da06145f0564d2894d167fdb5f.

File: z1_description/urdf/z1.ros2_control.xacro (robot description, xacro)
@@ -9,8 +9,8 @@
         params="
         name:='z1'
-        sim_ignition:=false
+        sim_ignition:=true
         sim_coppelia:=false
         prefix:=''
-        with_gripper:=false
+        with_gripper:=true
         ">
         <ros2_control name="${name}" type="system">
@@ -29,10 +29,10 @@
             <joint name="joint1">
                 <command_interface name="position">
-                    <param name="min">${joint1_PositionMin}</param>
-                    <param name="max">${joint1_PositionMax}</param>
+                    <param name="min"> ${joint1_PositionMin} </param>
+                    <param name="max"> ${joint1_PositionMax} </param>
                 </command_interface>
                 <command_interface name="effort">
-                    <param name="min">-${torqueMax}</param>
-                    <param name="max">${torqueMax}</param>
+                    <param name="min"> -${torqueMax} </param>
+                    <param name="max"> ${torqueMax} </param>
                 </command_interface>
                 <state_interface name="position" />
@@ -42,11 +42,11 @@
             <joint name="joint2">
                 <command_interface name="position">
-                    <param name="min">${joint2_PositionMin}</param>
-                    <param name="max">${joint2_PositionMax}</param>
+                    <param name="min"> ${joint2_PositionMin} </param>
+                    <param name="max"> ${joint2_PositionMax} </param>
                 </command_interface>
                 <command_interface
                     name="effort">
-                    <param name="min">-${torqueMax}</param>
-                    <param name="max">${torqueMax}</param>
+                    <param name="min"> -${torqueMax} </param>
+                    <param name="max"> ${torqueMax} </param>
                 </command_interface>
                 <xacro:if value="${sim_ignition}">
@@ -64,10 +64,10 @@
             <joint name="joint3">
                 <command_interface name="position">
-                    <param name="min">${joint3_PositionMin}</param>
-                    <param name="max">${joint3_PositionMax}</param>
+                    <param name="min"> ${joint3_PositionMin} </param>
+                    <param name="max"> ${joint3_PositionMax} </param>
                 </command_interface>
                 <command_interface name="effort">
-                    <param name="min">-${torqueMax}</param>
-                    <param name="max">${torqueMax}</param>
+                    <param name="min"> -${torqueMax} </param>
+                    <param name="max"> ${torqueMax} </param>
                 </command_interface>
                 <xacro:if value="${sim_ignition}">
@@ -85,10 +85,10 @@
             <joint name="joint4">
                 <command_interface name="position">
-                    <param name="min">${joint4_PositionMin}</param>
-                    <param name="max">${joint4_PositionMax}</param>
+                    <param name="min"> ${joint4_PositionMin} </param>
+                    <param name="max"> ${joint4_PositionMax} </param>
                 </command_interface>
                 <command_interface name="effort">
-                    <param name="min">-${torqueMax}</param>
-                    <param name="max">${torqueMax}</param>
+                    <param name="min"> -${torqueMax} </param>
+                    <param name="max"> ${torqueMax} </param>
                 </command_interface>
                 <state_interface name="position" />
@@ -98,10 +98,10 @@
             <joint name="joint5">
                 <command_interface name="position">
-                    <param name="min">${joint5_PositionMin}</param>
-                    <param name="max">${joint5_PositionMax}</param>
+                    <param name="min"> ${joint5_PositionMin} </param>
+                    <param name="max"> ${joint5_PositionMax} </param>
                 </command_interface>
                 <command_interface name="effort">
-                    <param name="min">-${torqueMax}</param>
-                    <param name="max">${torqueMax}</param>
+                    <param name="min"> -${torqueMax} </param>
+                    <param name="max"> ${torqueMax} </param>
                 </command_interface>
                 <state_interface name="position" />
@@ -111,10 +111,10 @@
             <joint name="joint6">
                 <command_interface name="position">
-                    <param name="min">${joint6_PositionMin}</param>
-                    <param name="max">${joint6_PositionMax}</param>
+                    <param name="min"> ${joint6_PositionMin} </param>
+                    <param name="max"> ${joint6_PositionMax} </param>
                 </command_interface>
                 <command_interface name="effort">
-                    <param name="min">-${torqueMax}</param>
-                    <param name="max">${torqueMax}</param>
+                    <param name="min"> -${torqueMax} </param>
+                    <param name="max"> ${torqueMax} </param>
                 </command_interface>
                 <state_interface name="position" />
@@ -125,10 +125,10 @@
                 <joint name="jointGripper">
                     <command_interface name="position">
-                        <param name="min">${Gripper_PositionMin}</param>
-                        <param name="max">${Gripper_PositionMax}</param>
+                        <param name="min"> ${Gripper_PositionMin} </param>
+                        <param name="max"> ${Gripper_PositionMax} </param>
                     </command_interface>
                     <command_interface name="effort">
-                        <param name="min">-${torqueMax}</param>
-                        <param name="max">${torqueMax}</param>
+                        <param name="min"> -${torqueMax} </param>
+                        <param name="max"> ${torqueMax} </param>
                     </command_interface>
                     <state_interface name="position" />

File: z1_description/urdf/z1.urdf.xacro (robot description, xacro)
@@ -106,5 +106,5 @@
     </link>
     <joint name="joint3" type="revolute">
-        <origin rpy="0 -0.1 0" xyz="-0.35 0 0" />
+        <origin rpy="0 0 0" xyz="-0.35 0 0" />
         <parent link="link02" />
         <child link="link03" />
@@ -306,6 +306,6 @@
         <gazebo reference="world" />
         <gazebo>
-            <!-- <plugin filename="libign_ros2_control-system.so" name="ign_ros2_control::IgnitionROS2ControlPlugin"> -->
-            <plugin filename="libgz_ros2_control-system.so" name="gz_ros2_control::GazeboSimROS2ControlPlugin">
+            <plugin filename="libign_ros2_control-system.so"
+                name="ign_ros2_control::IgnitionROS2ControlPlugin">
                 <parameters> $(arg controllers) </parameters>
                 <robot_param> robot_description </robot_param>
